File: hardware/nano-pcb/CellDoc-Nano.kicad_pcb (KiCad board)
At the start: 2 copper layers, 95 x 100 mm, 28 parts, among them J2 DS18B20 Zelle, J3 DS18B20 Last opt., J4 OLED opt., J5 QR GM861S opt., Q1 AO3400, Q2 AO3401, Q3 AO3400, Q4 AO3400, U1 ESP32-C3 SuperMini, U2 INA226 (Shunt R010), U3 TP4056 USB-C

Commit message: Nano-Platine: Beschriftung OLED und QR-Scanner
Co-Authored-By: Claude Opus 5.5 <noreply@anthropic.com>
Claude-Session: https://claude.ai/code/session_01WtJ5FLprrJxW2qKdxjRQsn
Other:
- board text added: "OLED"
- board text added: "QR-Scanner"
Changed lines of the file:
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@@
     (effects (font (size 0.8 0.8) (thickness 0.12)))
+  )
+  (gr_text "QR-Scanner" (at 47.9 68.6 90) (layer "F.SilkS")
+    (effects (font (size 0.8 0.8) (thickness 0.12)))
+  )
+  (gr_text "OLED" (at 48.8 63) (layer "F.SilkS")
+    (effects (font (size 0.9 0.9) (thickness 0.135)))
   )
   (gr_text "v1.1 · 2026-10" (at 57.5 76) (layer "F.SilkS")
